File: bt-rc-tx/bt-rc-tx.kicad_pcb (KiCad board)
At the start: 2 copper layers, 80 x 60 mm, 19 parts, among them J1 Battery 3V, J3 SW Debug, J4 Inhibit Shutdown, SW2 BUTTON1, SW3 BUTTON2, U2 STM32U031F8Px

Commit message: fixes
Routing:
- net GND: track 0.00 -> 19.6 mm, vias 0 -> 2
- net /LED1: track 38.8 -> 40.3 mm
Other:
- board text added: "${PROJECTNAME} Rev A"

Commit message: fixes
Parts:
- turned C1 to -90 degrees
Connections:
- J1 pad 1: +BATT -> GND
- J1 pad 2: GND -> +BATT
- J3 pad 1: +BATT -> GND
- J3 pad 2: GND -> +BATT
- J4 pad 1: /INH_SHDN -> GND
- J4 pad 2: GND -> /INH_SHDN
Routing:
- net Net-(U2-PA1/PA2): track 13.4 -> 19.9 mm
- net +BATT: track 112.5 -> 107.0 mm
- net Net-(U2-PA0): track 30.0 -> 28.0 mm
- net /INH_SHDN: track 37.7 -> 36.7 mm
- net GND: track 19.6 -> 20.2 mm
Other:
- board text added: "${PROJECTNAME} Rev A 2026-05-28"
- board text removed: "${PROJECTNAME} Rev A"
Changed lines of the file:
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@@
 	(paper "A4")
 	(title_block
-		(title "Bluetooth LE Remote Control Transmitteer")
+		(title "Bluetooth LE Remote Control Transmitter")
 		(date "2026-05-15")
 		(rev "A")
@@
 			(outputformat 1)
 			(mirror no)
-			(drillshape 1)
+			(drillshape 0)
 			(scaleselection 1)
-			(outputdirectory "")
+			(outputdirectory "/home/josef/projects/pico-pwrmgr-u031-01/bt-rc-tx/gerbers/")
 		)
 	)
@@
 	(footprint "Capacitor_SMD:C_1206_3216Metric"
 		(layer "F.Cu")
-		(at 131 96.475 90)
+		(at 131 96.475 -90)
 		(descr "Capacitor SMD 1206 (3216 Metric), square (rectangular) end terminal, IPC-7351 nominal, (Body size source: IPC-SM-782 page 76, https://www.pcb-3d.com/wordpress/wp-content/uploads/ipc-sm-782a_amendment_1_and_2.pdf)")
 		(tags "capacitor")
@@
 		)
 		(property "Value" "47u"
-			(at 0 1.85 90)
+			(at -1.475 2 90)
 			(layer "F.Fab")
 			(effects
@@
 		(duplicate_pad_numbers_are_jumpers no)
 		(fp_line
-			(start -0.711252 -0.91)
-			(end 0.711252 -0.91)
+			(start -0.711252 0.91)
+			(end 0.711252 0.91)
 			(stroke
 				(width 0.12)
@@
 		)
 		(fp_line
-			(start -0.711252 0.91)
-			(end 0.711252 0.91)
+			(start -0.711252 -0.91)
+			(end 0.711252 -0.91)
 			(stroke
 				(width 0.12)
@@
 		)
 		(pad "1" smd roundrect
-			(at -1.475 0 90)
+			(at -1.475 0 270)
 			(size 1.15 1.8)
 			(layers "F.Cu" "F.Mask" "F.Paste")
@@
 		)
 		(pad "2" smd roundrect
-			(at 1.475 0 90)
+			(at 1.475 0 270)
 			(size 1.15 1.8)
 			(layers "F.Cu" "F.Mask" "F.Paste")
@@
 			(layers "*.Cu" "*.Mask")
 			(remove_unused_layers no)
-			(net "+BATT")
+			(net "GND")
 			(pinfunction "Pin_1_1")
 			(pintype "power_out")
@@
 			(layers "*.Cu" "*.Mask")
 			(remove_unused_layers no)
-			(net "GND")
+			(net "+BATT")
 			(pinfunction "Pin_2_2")
 			(pintype "power_out")
@@
 			(layers "*.Cu" "*.Mask")
 			(remove_unused_layers no)
-			(net "/INH_SHDN")
+			(net "GND")
 			(pinfunction "Pin_1_1")
 			(pintype "passive")
@@
 			(layers "*.Cu" "*.Mask")
 			(remove_unused_layers no)
-			(net "GND")
+			(net "/INH_SHDN")
 			(pinfunction "Pin_2_2")
 			(pintype "passive")
@@
 			(layers "*.Cu" "*.Mask")
 			(remove_unused_layers no)
-			(net "+BATT")
+			(net "GND")
 			(pinfunction "Pin_1_1")
 			(pintype "passive")
@@
 			(layers "*.Cu" "*.Mask")
 			(remove_unused_layers no)
-			(net "GND")
+			(net "+BATT")
 			(pinfunction "Pin_2_2")
 			(pintype "passive")
@@
 	)
 	(gr_line
-		(start 136 53)
-		(end 136 69.5)
-		(stroke
-			(width 0.1)
-			(type default)
-		)
-		(layer "F.SilkS")
-	)
-	(gr_line
-		(start 136 92.5)
-		(end 136 109)
-		(stroke
-			(width 0.1)
-			(type default)
-		)
-		(layer "F.SilkS")
-	)
-	(gr_line
 		(start 85 55)
 		(end 85 107)
@@
 		(layer "Edge.Cuts")
 	)
-	(gr_text "${PROJECTNAME}\nRev A"
-		(at 148 107.5 0)
+	(gr_text "${PROJECTNAME}\nRev A\n2026-05-28"
+		(at 142.5 109 0)
 		(layer "F.SilkS")
 		(effects
@@
 	)
 	(segment
+		(start 131.45 97.5)
+		(end 131 97.95)
+		(width 0.2)
+		(layer "F.Cu")
+		(net "GND")
+	)
+	(segment
 		(start 91.775 77.725)
 		(end 91 78.5)
@@
 	)
 	(segment
-		(start 86 83)
-		(end 86 76.5)
+		(start 127.16 67.16)
+		(end 124.5 67.16)
 		(width 0.2)
 		(layer "F.Cu")
@@
 	)
 	(segment
-		(start 127.16 67.16)
-		(end 124.5 67.16)
+		(start 86.5 83.5)
+		(end 86.5 76)
+		(width 0.2)
+		(layer "F.Cu")
+		(net "+3.3V")
+	)
+	(segment
+		(start 88 85)
+		(end 86.5 83.5)
 		(width 0.2)
 		(layer "F.Cu")
@@
 	)
 	(segment
-		(start 86 76.5)
+		(start 86.5 76)
 		(end 87 75.5)
 		(width 0.2)
@@
 		(net "+3.3V")
 	)
-	(segment
-		(start 88 85)
-		(end 86 83)
-		(width 0.2)
-		(layer "F.Cu")
-		(net "+3.3V")
-	)
 	(via
 		(at 89.9 75.5)
@@
 	)
 	(segment
-		(start 128.5 60.5)
-		(end 127.54 59.54)
+		(start 129 95)
+		(end 131 95)
 		(width 0.2)
 		(layer "F.Cu")
@@
 	)
 	(segment
-		(start 135 97.5)
-		(end 131.45 97.5)
+		(start 95.5 78.5)
+		(end 96 79)
 		(width 0.2)
 		(layer "F.Cu")
@@
 	)
 	(segment
-		(start 131 97.95)
-		(end 129.45 97.95)
+		(start 128.5 60.5)
+		(end 127.54 59.54)
 		(width 0.2)
 		(layer "F.Cu")
@@
 	)
 	(segment
-		(start 95.5 78.5)
-		(end 96 79)
+		(start 135 64.08)
+		(end 129.08 64.08)
 		(width 0.2)
 		(layer "F.Cu")
@@
 	)
 	(segment
-		(start 124.5 59.54)
-		(end 127.04 59.54)
+		(start 127.54 59.54)
+		(end 124.5 59.54)
 		(width 0.2)
 		(layer "F.Cu")
@@
 	)
 	(segment
-		(start 128.5 97)
-		(end 128.5 67)
-		(width 0.2)
-		(layer "F.Cu")
-		(net "+BATT")
-	)
-	(segment
-		(start 128.88 66.62)
-		(end 128.5 66.24)
+		(start 129.08 64.08)
+		(end 128.5 63.5)
 		(width 0.2)
 		(layer "F.Cu")
@@
 	)
 	(segment
-		(start 135 66.62)
-		(end 128.88 66.62)
-		(width 0.2)
-		(layer "F.Cu")
-		(net "+BATT")
-	)
-	(segment
-		(start 128.5 60.5)
-		(end 128.5 67)
+		(start 96 80.5)
+		(end 96 79)
 		(width 0.2)
 		(layer "F.Cu")
@@
 	)
 	(segment
-		(start 96 80.5)
-		(end 96 79)
+		(start 128.5 94.5)
+		(end 129 95)
 		(width 0.2)
 		(layer "F.Cu")
@@
 	)
 	(segment
-		(start 129.45 97.95)
-		(end 128.5 97)
+		(start 100.5 71.4)
+		(end 95.5 76.4)
 		(width 0.2)
 		(layer "F.Cu")
@@
 	)
 	(segment
-		(start 100.5 71.4)
-		(end 95.5 76.4)
+		(start 131.04 94.96)
+		(end 131 95)
 		(width 0.2)
 		(layer "F.Cu")
@@
 	)
 	(segment
-		(start 131.45 97.5)
-		(end 131 97.95)
+		(start 128.5 94.5)
+		(end 128.5 63.5)
 		(width 0.2)
 		(layer "F.Cu")
@@
 	)
 	(segment
-		(start 127.54 59.54)
-		(end 124.5 59.54)
+		(start 96 79)
+		(end 95.375 78.375)
 		(width 0.2)
 		(layer "F.Cu")
@@
 	)
 	(segment
-		(start 96 79)
-		(end 95.375 78.375)
+		(start 135 94.96)
+		(end 131.04 94.96)
 		(width 0.2)
 		(layer "F.Cu")
@@
 	)
 	(segment
-		(start 128.5 66.24)
-		(end 128.5 66)
+		(start 95.375 78.375)
+		(end 93.1375 78.375)
 		(width 0.2)
 		(layer "F.Cu")
@@
 	)
 	(segment
-		(start 95.375 78.375)
-		(end 93.1375 78.375)
+		(start 128.5 63.5)
+		(end 128.5 60.5)
 		(width 0.2)
 		(layer "F.Cu")
@@
 	)
 	(segment
-		(start 87 77)
-		(end 86.5 77.5)
+		(start 87.5 77.5)
+		(end 88 77)
 		(width 0.2)
 		(layer "F.Cu")
@@
 	)
 	(segment
-		(start 87.125 81.625)
-		(end 93.1375 81.625)
+		(start 87.5 81)
+		(end 87.5 77.5)
 		(width 0.2)
 		(layer "F.Cu")
@@
 	)
 	(segment
-		(start 101 69.5)
+		(start 91.5 72.5)
 		(end 94.5 69.5)
 		(width 0.2)
@@
 	)
 	(segment
-		(start 91.5 75.5)
+		(start 88 77)
 		(end 90 77)
 		(width 0.2)
@@
 	)
 	(segment
-		(start 91.5 72.5)
-		(end 91.5 75.5)
+		(start 101 69.5)
+		(end 94.5 69.5)
 		(width 0.2)
 		(layer "F.Cu")
@@
 	)
 	(segment
-		(start 86.5 81)
-		(end 87.125 81.625)
+		(start 93.1375 81.625)
+		(end 88.125 81.625)
 		(width 0.2)
 		(layer "F.Cu")
@@
 	)
 	(segment
-		(start 86.5 77.5)
-		(end 86.5 81)
+		(start 90 77)
+		(end 91.5 75.5)
 		(width 0.2)
 		(layer "F.Cu")
@@
 	)
 	(segment
-		(start 94.5 69.5)
-		(end 91.5 72.5)
+		(start 88.125 81.625)
+		(end 87.5 81)
 		(width 0.2)
 		(layer "F.Cu")
@@
 	)
 	(segment
-		(start 90 77)
-		(end 87 77)
+		(start 91.5 75.5)
+		(end 91.5 72.5)
 		(width 0.2)
 		(layer "F.Cu")
@@
 	)
 	(segment
+		(start 101 92.5)
+		(end 94.5 92.5)
+		(width 0.2)
+		(layer "B.Cu")
+		(net "Net-(U2-PA1{slash}PA2)")
+	)
+	(segment
 		(start 100.175 80.325)
 		(end 101 79.5)
@@
 	)
 	(segment
-		(start 132.54 82.54)
-		(end 135 82.54)
+		(start 101 79.5)
+		(end 129.5 79.5)
 		(width 0.2)
 		(layer "B.Cu")
@@
 	)
 	(segment
-		(start 101 79.5)
-		(end 129.5 79.5)
+		(start 135 80)
+		(end 130 80)
 		(width 0.2)
 		(layer "B.Cu")
@@
 	)
 	(segment
-		(start 129.5 79.5)
-		(end 132.54 82.54)
+		(start 130 80)
+		(end 129.5 79.5)
 		(width 0.2)
 		(layer "B.Cu")
