File: bt-rc-tx/bt-rc-tx.kicad_sch (KiCad schematic)
At the start: 19 parts, among them J1 Battery 3V, J3 SW Debug, J4 Inhibit Shutdown, SW2 BUTTON1, SW3 BUTTON2, U2 STM32U031F8Px

Commit message: fixes
Connections:
- net +BATT: now also J1.2 (Pin_2), J3.2 (Pin_2); no longer J1.1 (Pin_1), J3.1 (Pin_1)
- net GND: now also J1.1 (Pin_1), J3.1 (Pin_1), J4.1 (Pin_1); no longer J1.2 (Pin_2), J3.2 (Pin_2), J4.2 (Pin_2)
- net INH_SHDN: now also J4.2 (Pin_2); no longer J4.1 (Pin_1)
Other:
- moved on the sheet: J4
